Commit message: collisionmir

File: src/python/models/robotiq_box.urdf (robot description, URDF)
Before this commit: robot box_hand, 1 links, 0 joints
Links:
- link box_hand_1: geometry collision box size=0.1 0.1 0.1; visual box size=0.1 0.1 0.1
Joints:
- added joint planar_joint: type planar, parent world, child box_hand_1, axis 0 1 0
